File: PCB/ESP32_Board/ESP32_Board.kicad_pcb (KiCad board)
At the start: 2 copper layers, 4 parts, among them U1 ESP32-S3-DevKitC

Commit message: 1
Parts:
- moved C1 154.0 mm to (1.07, 37.4), turned to 0 degrees
- moved R1 132.1 mm to (1.04, 44.1)
- moved U1 132.1 mm to (-29.4, 43.3)
- moved C2 111.2 mm to (1.07, 40.7)
Routing:
- net (no net): vias 0 -> 39

Commit message: 3
Parts:
- added D1: D_Small, Diode_SMD:D_SMA, B.Cu at (93.5, 51.0)
- added K1: SANYOU_SRD_Form_C, Relay_THT:Relay_SPDT_SANYOU_SRD_Series_Form_C, F.Cu at (98.5, 55.0)
- added Q1: Q_NPN_BCE, Package_TO_SOT_SMD:SOT-89-3_Handsoldering, B.Cu at (94.4, 61.0)
- added R2: R_Small, Resistor_SMD:R_1206_3216Metric_Pad1.30x1.75mm_HandSolder, B.Cu at (89.4, 61.0)
- added U2: PC817, Package_DIP:DIP-4_W7.62mm, F.Cu at (100.4, 80.4)
- R1: moved to B.Cu
- moved R1 90.8 mm to (90.8, 57.1)
- moved C1 65.4 mm to (66.1, 44.5)
- moved C2 65.4 mm to (66.1, 47.8)
- moved U1 65.4 mm to (35.6, 50.4)
Connections:
- R1 pad 1: unconnected-(R1-Pad1) -> RELAY_LAZER
- R1 pad 2: unconnected-(R1-Pad2) -> Net-(Q1-B)
Routing:
- net (no net): vias 39 -> 0
