File: PCB/ESP32_Board/ESP32_Board.kicad_sch (KiCad schematic)
At the start: 4 parts, among them U1 ESP32-S3-DevKitC

Commit message: 3
Parts:
- added D1, D2, D3: D_Small, Diode_SMD:D_SMA, symbol Device:D_Small
- added J1: Conn_01x02, symbol Connector_Generic:Conn_01x02
- added J2, J3, J4: Conn_01x03, symbol Connector_Generic:Conn_01x03
- added K1, K2, K3: SANYOU_SRD_Form_C, Relay_THT:Relay_SPDT_SANYOU_SRD_Series_Form_C, symbol Relay:SANYOU_SRD_Form_C
- added Q1, Q2, Q3: Q_NPN_BCE, Package_TO_SOT_SMD:SOT-89-3_Handsoldering, symbol Device:Q_NPN_BCE
- added Q4: IRF740, Package_TO_SOT_THT:TO-220-3_Vertical, symbol Transistor_FET:IRF740
- added R10, R11, R2, R3, R4, R5, R6, R7, R8: R_Small, Resistor_SMD:R_1206_3216Metric_Pad1.30x1.75mm_HandSolder, symbol Device:R_Small
- added U2: PC817, Package_DIP:DIP-4_W7.62mm, symbol Isolator:PC817
Connections:
- net 5V: now also D1.1 (K), D2.1 (K), D3.1 (K), K1.5, K2.5, K3.5
- net GND: now also J2.2 (Pin_2), J3.2 (Pin_2), Q1.3 (E), Q2.3 (E), Q3.3 (E), Q4.3 (S), R11.1, R2.2, R4.2, R6.2, R8.1, U2.2
- net RELAY_LAZER: now reaches R1.1
- net RELAY_LAZER: now also R2.1
- net at R1.2: now also Q1.1 (B)
- new net: D1.2 (A), K1.2, Q1.2 (C)
- new net: J3.1 (Pin_1), K2.1
- new net: D2.2 (A), K2.2, Q2.2 (C)
- new net: Q3.1 (B), R5.2
- new net: J2.1 (Pin_1), K1.1
- new net: R10.2, R11.2
- new net: Q2.1 (B), R3.2
- new net: R7.1, R8.2, U2.3
- new net: Q4.1 (G), R7.2
- new net: J1.2 (Pin_2), Q4.2 (D)
- new net: D3.2 (A), K3.2, Q3.2 (C)
- new net: R10.1, U2.1
- new net: J4.1 (Pin_1), K3.3
- new net: J4.2 (Pin_2), K3.1
- new net: J4.3 (Pin_3), K3.4
- new net 12V: J1.1 (Pin_1), K1.3, K2.3, U2.4
- new net LAZER_PWM: J2.3 (Pin_3)
- new net PWM_VACCUM: J3.3 (Pin_3)
- new net RELAY_COMPRESSOR: R5.1, R6.1
- new net RELAY_VACCUM: R3.1, R4.1
